Commit message: ✨

File: reachy_mobile_description/urdf/reachy_mobile.urdf (robot description, URDF)
Before this commit: robot reachy_mobile, 32 links, 31 joints
Links:
- link base_link: geometry collision mesh filename=package://reachy_mobile_description/meshes/simplify_starter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 scale=0.001 0.001 0.001; visual mesh filename=package://reachy_mobile_description/meshes/starter_kit.stl scale=0.001 0.001 0.001

File: reachy_mobile_description/urdf/swd_starter_kit.urdf (robot description, URDF)
Before this commit: robot swd_starter_kit, 4 links, 3 joints
Links:
- link base_link: geometry collision mesh filename=package://reachy_mobile_description/meshes/simplify_starter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 scale=0.001 0.001 0.001; visual mesh filename=package://reachy_mobile_description/meshes/starter_kit.stl scale=0.001 0.001 0.001
